File: ASIC-simulator/tt04-fpga-ICE40UP5k/breakout-fpga-ICE40UP5K.kicad_sch (KiCad schematic)
At the start: 92 parts, among them J1 USB_C, J2 Conn_02x04_Odd_Even, SW1 434121025816, SW2 434121025816, SW3 434121025816, U1 AP2112K-3.3, U2 AP2112K-1.2, U3 ICE40UP5K-SG48ITR, U4 W25Q32JVSS, X1 24MHz

Commit message: Final DNPs used
Parts:
- C23, R17, R20, R30, SW3: now not fitted
- R28: now fitted
Changed lines of the file:
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@@
 	(title_block
 		(title "TT04+ FPGA ASIC Simulator ")
-		(date "2024-04-06")
-		(rev "1.0")
+		(date "2024-04-24")
+		(rev "1.1")
 		(company "Psychogenic Technologies ")
 		(comment 1 "(C) 2024 Pat Deegan")
@@
 		(in_bom yes)
 		(on_board yes)
-		(dnp no)
+		(dnp yes)
 		(fields_autoplaced yes)
 		(property "Reference" "R30"
@@
 			)
 		)
+		(property "Variant" ""
+			(at 205.74 36.83 0)
+			(effects
+				(font
+					(size 1.27 1.27)
+				)
+				(hide yes)
+			)
+		)
 		(pin "2"
 		)
@@
 		(in_bom yes)
 		(on_board yes)
-		(dnp no)
+		(dnp yes)
 		(fields_autoplaced yes)
 		(property "Reference" "R17"
@@
 		(in_bom yes)
 		(on_board yes)
-		(dnp no)
+		(dnp yes)
 		(fields_autoplaced yes)
 		(property "Reference" "C23"
@@
 		(in_bom yes)
 		(on_board yes)
-		(dnp no)
+		(dnp yes)
 		(fields_autoplaced yes)
 		(property "Reference" "R20"
@@
 			)
 		)
+		(property "Variant" ""
+			(at 243.84 231.14 0)
+			(effects
+				(font
+					(size 1.27 1.27)
+				)
+				(hide yes)
+			)
+		)
 		(pin "1"
 		)
@@
 		(in_bom yes)
 		(on_board yes)
-		(dnp yes)
+		(dnp no)
 		(fields_autoplaced yes)
 		(property "Reference" "R28"
@@
 		(in_bom yes)
 		(on_board yes)
-		(dnp no)
+		(dnp yes)
 		(property "Reference" "SW3"
 			(at 234.95 221.996 90)
