File: breakout-tt06-qfn/analog_connectors.kicad_sch (KiCad schematic)
At the start: 12 parts, among them J10 U.FL, J11 U.FL, J12 U.FL, J13 U.FL, J8 U.FL, J9 U.FL

Commit message: TT06 carrier v1.1 as in production run
Parts:
- J10, J11, J12, J13, J8, J9: Characteristics (none) -> ipex/u.fl connector
