File: breakout-qfn/analog_connectors.kicad_sch (KiCad schematic)
At the start: 12 parts, among them J10 U.FL, J11 U.FL, J12 U.FL, J13 U.FL, J8 U.FL, J9 U.FL

Commit message: refactor, tt07
Other:
- title: (none) -> Analog Pin Breakouts
Changed lines of the file:
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@@
 	(generator "eeschema")
 	(generator_version "8.0")
-	(paper "A4")
+	(paper "User" 150 160)
+	(title_block
+		(title "Analog Pin Breakouts")
+		(date "2024-12-10")
+		(rev "2.0")
+	)
 	(junction
 		(at 68.58 64.77)
@@
 		)
 		(instances
-			(project "breakout-tt06-qfn"
+			(project "breakout-tt07-qfn"
 				(path "/b38c65ac-2d57-46f9-9a32-ad09573ee400/a4870ec5-4ad2-4ab2-a570-743ccf31c608"
 					(reference "#PWR068")
@@
 		)
 		(instances
-			(project "breakout-tt06-qfn"
+			(project "breakout-tt07-qfn"
 				(path "/b38c65ac-2d57-46f9-9a32-ad09573ee400/a4870ec5-4ad2-4ab2-a570-743ccf31c608"
 					(reference "JP11")
@@
 		)
 		(instances
-			(project "breakout-tt06-qfn"
+			(project "breakout-tt07-qfn"
 				(path "/b38c65ac-2d57-46f9-9a32-ad09573ee400/a4870ec5-4ad2-4ab2-a570-743ccf31c608"
 					(reference "#PWR072")
@@
 		)
 		(instances
-			(project "breakout-tt06-qfn"
+			(project "breakout-tt07-qfn"
 				(path "/b38c65ac-2d57-46f9-9a32-ad09573ee400/a4870ec5-4ad2-4ab2-a570-743ccf31c608"
 					(reference "#PWR071")
@@
 		)
 		(instances
-			(project "breakout-tt06-qfn"
+			(project "breakout-tt07-qfn"
 				(path "/b38c65ac-2d57-46f9-9a32-ad09573ee400/a4870ec5-4ad2-4ab2-a570-743ccf31c608"
 					(reference "J11")
@@
 		)
 		(instances
-			(project "breakout-tt06-qfn"
+			(project "breakout-tt07-qfn"
 				(path "/b38c65ac-2d57-46f9-9a32-ad09573ee400/a4870ec5-4ad2-4ab2-a570-743ccf31c608"
 					(reference "JP9")
@@
 		)
 		(instances
-			(project "breakout-tt06-qfn"
+			(project "breakout-tt07-qfn"
 				(path "/b38c65ac-2d57-46f9-9a32-ad09573ee400/a4870ec5-4ad2-4ab2-a570-743ccf31c608"
 					(reference "JP7")
@@
 		)
 		(instances
-			(project "breakout-tt06-qfn"
+			(project "breakout-tt07-qfn"
 				(path "/b38c65ac-2d57-46f9-9a32-ad09573ee400/a4870ec5-4ad2-4ab2-a570-743ccf31c608"
 					(reference "J13")
@@
 		)
 		(instances
-			(project "breakout-tt06-qfn"
+			(project "breakout-tt07-qfn"
 				(path "/b38c65ac-2d57-46f9-9a32-ad09573ee400/a4870ec5-4ad2-4ab2-a570-743ccf31c608"
 					(reference "J9")
@@
 		)
 		(instances
-			(project "breakout-tt06-qfn"
+			(project "breakout-tt07-qfn"
 				(path "/b38c65ac-2d57-46f9-9a32-ad09573ee400/a4870ec5-4ad2-4ab2-a570-743ccf31c608"
 					(reference "#PWR070")
@@
 		)
 		(instances
-			(project "breakout-tt06-qfn"
+			(project "breakout-tt07-qfn"
 				(path "/b38c65ac-2d57-46f9-9a32-ad09573ee400/a4870ec5-4ad2-4ab2-a570-743ccf31c608"
 					(reference "JP12")
@@
 		)
 		(instances
-			(project "breakout-tt06-qfn"
+			(project "breakout-tt07-qfn"
 				(path "/b38c65ac-2d57-46f9-9a32-ad09573ee400/a4870ec5-4ad2-4ab2-a570-743ccf31c608"
 					(reference "JP8")
@@
 		)
 		(instances
-			(project "breakout-tt06-qfn"
+			(project "breakout-tt07-qfn"
 				(path "/b38c65ac-2d57-46f9-9a32-ad09573ee400/a4870ec5-4ad2-4ab2-a570-743ccf31c608"
 					(reference "#PWR073")
@@
 		)
 		(instances
-			(project "breakout-tt06-qfn"
+			(project "breakout-tt07-qfn"
 				(path "/b38c65ac-2d57-46f9-9a32-ad09573ee400/a4870ec5-4ad2-4ab2-a570-743ccf31c608"
 					(reference "JP10")
@@
 		)
 		(instances
-			(project "breakout-tt06-qfn"
+			(project "breakout-tt07-qfn"
 				(path "/b38c65ac-2d57-46f9-9a32-ad09573ee400/a4870ec5-4ad2-4ab2-a570-743ccf31c608"
 					(reference "#PWR069")
@@
 		)
 		(instances
-			(project "breakout-tt06-qfn"
+			(project "breakout-tt07-qfn"
 				(path "/b38c65ac-2d57-46f9-9a32-ad09573ee400/a4870ec5-4ad2-4ab2-a570-743ccf31c608"
 					(reference "J12")
@@
 		)
 		(instances
-			(project "breakout-tt06-qfn"
+			(project "breakout-tt07-qfn"
 				(path "/b38c65ac-2d57-46f9-9a32-ad09573ee400/a4870ec5-4ad2-4ab2-a570-743ccf31c608"
 					(reference "J10")
@@
 		)
 		(instances
-			(project "breakout-tt06-qfn"
+			(project "breakout-tt07-qfn"
 				(path "/b38c65ac-2d57-46f9-9a32-ad09573ee400/a4870ec5-4ad2-4ab2-a570-743ccf31c608"
 					(reference "J8")
