File: breakout-qfn/breakout-tt07-qfn.kicad_pcb (KiCad board)
At the start: 2 copper layers, 50 x 52 mm, 153 parts, among them J1 Conn_01x04, J10 U.FL, J11 U.FL, J12 U.FL, J13 U.FL, J2 U.FL, J3 U.FL, J4 U.FL, J5 U.FL, J6 U.FL, J7 U.FL, J8 U.FL, J9 U.FL, U1 Openframe_QFN_TT06_REV2, U2 24LC02

Commit message: refactor, tt07
Connections:
- U2 pad 9: GND -> (no net)
Routing:
- net /c_sel_inc: track 54.1 -> 52.6 mm
- net /c_ena: track 39.1 -> 40.4 mm
- net /hd_c_rst_n: track 44.0 -> 44.8 mm
- net /uio1: track 33.0 -> 33.8 mm
- net vdda_all: vias 9 -> 10
Other:
- board text added: "IO PINS"
- board text added: "TT RUN 07"
- board text added: "clk"
- board text added: "i* : input io*: bidir o* : output"
- board text added: "i0"
- board text added: "i1"
- board text added: "i2"
- board text added: "i3"
- board text added: "i4"
- board text added: "i5"
- board text added: "i6"
- board text added: "i7"
- board text added: "io0"
- board text added: "io1"
- board text added: "io2"
- board text added: "io3"
- board text added: "io4"
- board text added: "io5"
- board text added: "io6"
- board text added: "io7"
- board text added: "o0"
- board text added: "o1"
- board text added: "o2"
- board text added: "o3"
- board text added: "o4"
- board text added: "o5"
- board text added: "o6"
- board text added: "o7"
- board text added: "~{rst}"
- board text removed: "TT RUN 06"
- board text removed: "bi0"
- board text removed: "bi1"
- board text removed: "bi2"
- board text removed: "bi3"
- board text removed: "bi4"
- board text removed: "bi5"
- board text removed: "bi6"
- board text removed: "bi7"
- board text removed: "in0"
- board text removed: "in1"
- board text removed: "in2"
- board text removed: "in3"
- board text removed: "in4"
- board text removed: "in5"
- board text removed: "in6"
- board text removed: "in7"
- board text removed: "out0"
- board text removed: "out1"
- board text removed: "out2"
- board text removed: "out3"
- board text removed: "out4"
- board text removed: "out5"
- board text removed: "out6"
- board text removed: "out7"
- board text removed: "pclk"
- board text removed: "p~{rst}"
