File: breakout-qfn/breakout-tt07-qfn.kicad_sch (KiCad schematic)
At the start: 42 parts, among them J1 Conn_01x04, U1 Openframe_QFN_TT06_REV2, U2 24LC02

Commit message: refactor, tt07
Other:
- title: TT06 Openframe breakout -> TT07 Openframe breakout
