File: breakout-ihp-qfn/breakout-ihp-qfn.kicad_pcb (KiCad board)
At the start: 4 copper layers, 50 x 50 mm, 114 parts, among them J1 Conn_01x12, J2 DF12NB-60DS-0.5V_51, J3 DF12NB-50DS-0.5V_51, U1 AP2112K-1.2, U2 AP2112K-1.8, U3 TT_IHP_ASIC, U4 24LC02

Commit message: More better and IPCish footprint for IHP
Parts:
- U3: footprint TinyTapeout:QFN-64-1EP_9x9mm_P0.5mm_EP4.7x4.7mm_IHP -> TinyTapeout:QFN-64-1EP_9x9mm_P0.5mm_EP4.7x4.7mm_IHP_B
- moved STITCHEP01 0.20 mm to (138.2, 77.3)
Routing:
- net GND: track 255.2 -> 261.9 mm
- net VDD_{IO}: track 141.1 -> 140.3 mm
- net VAA: track 81.7 -> 82.2 mm
