File: breakout-ihp-qfn/breakout-ihp-qfn.kicad_pcb (KiCad board)
At the start: 4 copper layers, 50 x 50 mm, 114 parts, among them J1 Conn_01x12, J2 DF12NB-60DS-0.5V_51, J3 DF12NB-50DS-0.5V_51, U1 AP2112K-1.2, U2 AP2112K-1.8, U3 TT_IHP_ASIC, U4 24LC02

Commit message: IHP breakout w/tnt footprint
Parts:
- U3: footprint TinyTapeout:QFN-64-1EP_9x9mm_P0.5mm_EP4.7x4.7mm_IHP_B -> TinyTapeout:QFN-64-1EP_9x9mm_P0.5mm_EP4.7x4.7mm_IHP_C
- moved LOGOIHP 0.25 mm to (148.4, 86.7)
Routing:
- net GND: track 261.9 -> 259.1 mm
- net VDD_{IO}: track 140.3 -> 141.3 mm
- net VAA: track 82.2 -> 83.0 mm
- net VDD_{CORE}: track 67.8 -> 68.5 mm

Commit message: fix off by one error
Parts:
- U3: footprint TinyTapeout:QFN-64-1EP_9x9mm_P0.5mm_EP4.7x4.7mm_IHP_C -> IHP-fp:QFN-64-1EP_9x9mm_P0.5mm_EP4.7x4.7mm_IHP_fuckedup
Routing:
- net GND: track 259.1 -> 264.4 mm, vias 79 -> 78
- net /increment: track 66.4 -> 65.2 mm
- net /uio1: track 25.6 -> 24.6 mm
- net /enable: track 95.3 -> 94.5 mm
- net /uio2: track 26.7 -> 25.9 mm
- net VDD_{CORE}: track 68.5 -> 69.3 mm, vias 6 -> 7
- net VDD_{IO}: track 141.3 -> 142.0 mm, vias 12 -> 13
- net /uio3: track 24.4 -> 23.7 mm
- net /rst_n: track 70.6 -> 69.9 mm
- net /uio4: track 25.1 -> 24.5 mm
- net /p_clk: track 23.2 -> 22.7 mm
Other:
- board text added: "TTIHP25b"
