File: breakout-ihp-qfn/breakout-ihp-qfn.kicad_sch (KiCad schematic)
At the start: 43 parts, among them J1 Conn_01x12, J2 DF12NB-60DS-0.5V_51, J3 DF12NB-50DS-0.5V_51, U1 AP2112K-1.2, U2 AP2112K-1.8, U3 TT_IHP_ASIC, U4 24LC02

Commit message: More better and IPCish footprint for IHP
Parts:
- U3: footprint TinyTapeout:QFN-64-1EP_9x9mm_P0.5mm_EP4.7x4.7mm_IHP -> TinyTapeout:QFN-64-1EP_9x9mm_P0.5mm_EP4.7x4.7mm_IHP_B

Commit message: IHP breakout w/tnt footprint
Parts:
- U3: footprint TinyTapeout:QFN-64-1EP_9x9mm_P0.5mm_EP4.7x4.7mm_IHP_B -> TinyTapeout:QFN-64-1EP_9x9mm_P0.5mm_EP4.7x4.7mm_IHP_C
