File: breakout-dip-gf/breakout-dip-gf.kicad_sch (KiCad schematic)
At the start: 39 parts, among them J1 USB_C, SW1 434121025816, U1 TT_GF_COB, U2 CH32X035G8U6, U3 AP2112K-3.3

Commit message: DIP component tweaks
Parts:
- C1, C2: JLC C23829972 -> C52923; LCSC C5673 -> (none); MPN GRM188D72A105KE01D -> CL05A105KA5NQNC
Changed lines of the file:
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@@
 			)
 		)
-		(property "MPN" "GRM188D72A105KE01D"
+		(property "MPN" "CL05A105KA5NQNC"
 			(at 82.55 33.02 0)
 			(hide yes)
@@
 			)
 		)
-		(property "LCSC" "C5673"
+		(property "LCSC" ""
 			(at 82.55 33.02 0)
 			(hide yes)
@@
 			)
 		)
-		(property "JLC" "C23829972"
+		(property "JLC" "C52923"
 			(at 82.55 33.02 0)
 			(hide yes)
@@
 			)
 		)
-		(property "MPN" "GRM188D72A105KE01D"
+		(property "MPN" "CL05A105KA5NQNC"
 			(at 73.66 33.02 0)
 			(hide yes)
@@
 			)
 		)
-		(property "LCSC" "C5673"
+		(property "LCSC" ""
 			(at 73.66 33.02 0)
 			(hide yes)
@@
 			)
 		)
-		(property "JLC" "C23829972"
+		(property "JLC" "C52923"
 			(at 73.66 33.02 0)
 			(hide yes)

Commit message: remap/reroute of pclk and VAA to Vcore
Parts:
- R6: now fitted
Connections:
- net VDD_{CORE}: now also R6.1
- net VIO_{REG}: no longer R6.1
- net p_clk: now also U2.8 (PA3); no longer U2.10 (PA5)
- net uin0: now also U2.14 (PB3); no longer U2.15 (PB4)
- net uio7: now also U2.21 (PB10)
- no-connect marks 3 -> 15

Commit message: bonding fids, silk markings, v1.0
Parts:
- C1, C2: Characteristics 1u 10V XR 0603 -> 1u 10V XR 0402
- C17, C19: Characteristics CAP CER 10UF 10V X5R 0603 -> 1u 10V XR 0603
- CONN1: renamed from C3; Characteristics (none) -> CONN SOCKET 32P
- R4, R5, R6: Characteristics RES SMD 0 OHM JUMPER 0805 -> RES SMD 0 OHM JUMPER 0402
- R7: Characteristics RES SMD 0 OHM JUMPER 1/10W 0603 -> RES SMD 0 OHM JUMPER 0402
- U1: Characteristics (none) -> TT GF ASIC
- U2: Characteristics (none) -> CH32X035 MCU
Other:
- note added: "32P DIP connector"
- note added: "Bridge Core and Analog Supplies"
- note added: "Bridge I/O and Core Supplies"
- note added: "DIP breakout for TinyTapeout GF180 ASICs"
- note added: "Supply chip with VUSB regulator output"
- note added: "TT-DIP firmware"
- note added: "This breakout allows direct access to the wire-bonded ASIC through the I/O, MUX and power pins. When used in conjunction with the , the system may be configured to automatically setup and clock specific designs on power-up, may do automatic detection of externally driven project MUX or clock/reset, and provides a Serial TUI interface through USB, for use by commander or directly through serial po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"
- note added: "https://github.com/psychogenic/TT-DIP"
- moved on the sheet: R4, R5, R6

Commit message: CoB DIP, as panelized
Parts:
- added J2, J3: (no value), TinyTapeout:PinHeader_1x16_P2.54mm_Placeholder, symbol TinyTapeout:DIP_Pinheader
Changed lines of the file:
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@@
 	)
 	(symbol
+		(lib_id "TinyTapeout:DIP_Pinheader")
+		(at 270.51 157.48 90)
+		(unit 1)
+		(body_style 1)
+		(exclude_from_sim no)
+		(in_bom yes)
+		(on_board yes)
+		(in_pos_files yes)
+		(dnp no)
+		(fields_autoplaced yes)
+		(property "Reference" "J3"
+			(at 271.78 157.4799 90)
+			(show_name no)
+			(do_not_autoplace no)
+			(effects
+				(font
+					(size 1.27 1.27)
+				)
+				(justify right)
+			)
+		)
+		(property "Value" ""
+			(at 270.51 157.48 0)
+			(show_name no)
+			(do_not_autoplace no)
+			(effects
+				(font
+					(size 1.27 1.27)
+				)
+			)
+		)
+		(property "Footprint" "TinyTapeout:PinHeader_1x16_P2.54mm_Placeholder"
+			(at 270.51 157.48 0)
+			(hide yes)
+			(show_name no)
+			(do_not_autoplace no)
+			(effects
+				(font
+					(size 1.27 1.27)
+				)
+			)
+		)
+		(property "Datasheet" ""
+			(at 270.51 157.48 0)
+			(hide yes)
+			(show_name no)
+			(do_not_autoplace no)
+			(effects
+				(font
+					(size 1.27 1.27)
+				)
+			)
+		)
+		(property "Description" ""
+			(at 270.51 157.48 0)
+			(hide yes)
+			(show_name no)
+			(do_not_autoplace no)
+			(effects
+				(font
+					(size 1.27 1.27)
+				)
+			)
+		)
+		(property "Characteristics" "1x16P 2.54mm Through Hole Plugin,P=2.54mm Pin Headers "
+			(at 270.51 157.48 90)
+			(hide yes)
+			(show_name no)
+			(do_not_autoplace no)
+			(effects
+				(font
+					(size 1.27 1.27)
+				)
+			)
+		)
+		(property "JLC" "C2894939"
+			(at 270.51 157.48 90)
+			(hide yes)
+			(show_name no)
+			(do_not_autoplace no)
+			(effects
+				(font
+					(size 1.27 1.27)
+				)
+			)
+		)
+		(property "LCSC" "C2894939"
+			(at 270.51 157.48 90)
+			(hide yes)
+			(show_name no)
+			(do_not_autoplace no)
+			(effects
+				(font
+					(size 1.27 1.27)
+				)
+			)
+		)
+		(property "MPN" "PZ254-1-16-Z-8.5"
+			(at 270.51 157.48 90)
+			(hide yes)
+			(show_name no)
+			(do_not_autoplace no)
+			(effects
+				(font
+					(size 1.27 1.27)
+				)
+			)
+		)
+		(instances
+			(project "breakout-dip-gf"
+				(path "/c110e856-5eae-4e29-a5dc-1f27e18e072d"
+					(reference "J3")
+					(unit 1)
+				)
+			)
+		)
+	)
+	(symbol
 		(lib_id "power:+3V3")
 		(at 45.72 147.32 0)
@@
 	)
 	(symbol
+		(lib_id "TinyTapeout:DIP_Pinheader")
+		(at 264.16 157.48 180)
+		(unit 1)
+		(body_style 1)
+		(exclude_from_sim no)
+		(in_bom yes)
+		(on_board yes)
+		(in_pos_files yes)
+		(dnp no)
+		(fields_autoplaced yes)
+		(property "Reference" "J2"
+			(at 265.43 157.4799 0)
+			(show_name no)
+			(do_not_autoplace no)
+			(effects
+				(font
+					(size 1.27 1.27)
+				)
+				(justify right)
+			)
+		)
+		(property "Value" ""
+			(at 264.16 157.48 0)
+			(show_name no)
+			(do_not_autoplace no)
+			(effects
+				(font
+					(size 1.27 1.27)
+				)
+			)
+		)
+		(property "Footprint" "TinyTapeout:PinHeader_1x16_P2.54mm_Placeholder"
+			(at 264.16 157.48 0)
+			(hide yes)
+			(show_name no)
+			(do_not_autoplace no)
+			(effects
+				(font
+					(size 1.27 1.27)
+				)
+			)
+		)
+		(property "Datasheet" ""
+			(at 264.16 157.48 0)
+			(hide yes)
+			(show_name no)
+			(do_not_autoplace no)
+			(effects
+				(font
+					(size 1.27 1.27)
+				)
+			)
+		)
+		(property "Description" ""
+			(at 264.16 157.48 0)
+			(hide yes)
+			(show_name no)
+			(do_not_autoplace no)
+			(effects
+				(font
+					(size 1.27 1.27)
+				)
+			)
+		)
+		(property "Characteristics" "1x16P 2.54mm Through Hole Plugin,P=2.54mm Pin Headers "
+			(at 264.16 157.48 0)
+			(hide yes)
+			(show_name no)
+			(do_not_autoplace no)
+			(effects
+				(font
+					(size 1.27 1.27)
+				)
+			)
+		)
+		(property "JLC" "C2894939"
+			(at 264.16 157.48 0)
+			(hide yes)
+			(show_name no)
+			(do_not_autoplace no)
+			(effects
+				(font
+					(size 1.27 1.27)
+				)
+			)
+		)
+		(property "LCSC" "C2894939"
+			(at 264.16 157.48 0)
+			(hide yes)
+			(show_name no)
+			(do_not_autoplace no)
+			(effects
+				(font
+					(size 1.27 1.27)
+				)
+			)
+		)
+		(property "MPN" "PZ254-1-16-Z-8.5"
+			(at 264.16 157.48 0)
+			(hide yes)
+			(show_name no)
+			(do_not_autoplace no)
+			(effects
+				(font
+					(size 1.27 1.27)
+				)
+			)
+		)
+		(instances
+			(project "breakout-dip-gf"
+				(path "/c110e856-5eae-4e29-a5dc-1f27e18e072d"
+					(reference "J2")
+					(unit 1)
+				)
+			)
+		)
+	)
+	(symbol
 		(lib_id "power:GND")
 		(at 82.55 35.56 0)
@@
 		(in_bom no)
 		(on_board yes)
-		(in_pos_files yes)
+		(in_pos_files no)
 		(dnp no)
 		(property "Reference" "CONN1"

Commit message: docs and prettyfication
Parts:
- J2, J3: value (none) -> PZ254-1-16-Z-8.5
Connections:
- no-connect marks 15 -> 17
Other:
- note added: "32P footprint DIP-32_W15.24mm"
- note added: "ASIC"
- note added: "BOOT"
- note added: "Hold BOOT button during power-up to put into firmware update mode and upgrade over USB"
- note added: "MCU"
- note added: "Regulated supply"
- note added: "Should be possible to upload firmware through USB but these allow pogo pins direct access to CH32 prog port."
- note removed: "Core Voltage Selection"
- note removed: "Options for basic filtering and ESD on USB conn. At a min, populate the ferrite and TVS diodes."
- note removed: "VDDIO SUPPLY"
- moved on the sheet: C1, C14, C15, C17, C18, C19, C2, C4, C5, C6, CONN1, FB1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
