File: breakout-gf-cob/breakout-gf-cob.kicad_pcb (KiCad board)
At the start: 4 copper layers, 50 x 50 mm, 109 parts, among them J1 Conn_01x12, J2 DF12NB-60DS-0.5V_51, J3 DF12NB-50DS-0.5V_51, U1 AP2112K-3.3, U2 AP2112K-3.3, U3 TT_GF_0p2_ASIC, U4 24LC02

Commit message: prep for prod
Other:
- board text added: "GF0p3 COB breakout v${REVISION}"
- board text removed: "GF26a COB breakout v${REVISION}"
