File: breakout-gf-cob/breakout-gf-cob.kicad_sch (KiCad schematic)
At the start: 43 parts, among them J1 Conn_01x12, J2 DF12NB-60DS-0.5V_51, J3 DF12NB-50DS-0.5V_51, U1 AP2112K-3.3, U2 AP2112K-3.3, U3 TT_GF_0p2_ASIC, U4 24LC02

Commit message: prep for prod
Parts:
- C1, C2, C5, C6: Characteristics 1u 10V XR 0603 -> 10u 10V XR 0603; LCSC (none) -> C19702; MPN (none) -> CL10A106KP8NNNC
- C10, C11, C12, C13, C14, C16, C17: LCSC (none) -> C52923; MPN CL05A105KO5NNNC -> CL05A105KA5NQNC
- R2: LCSC (none) -> C21189; MPN CRG0603ZR -> 0603WAF0000T5E
- R3, R6, R7: LCSC C95177 -> C21189; MPN CRG0603ZR -> 0603WAF0000T5E
- R4, R8, R9: LCSC C4143065 -> C17477; MPN RC0805JR-100RL -> 0805W8F0000T5E
Changed lines of the file:
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@@
 			)
 		)
-		(property "MPN" "CL05A105KO5NNNC"
+		(property "MPN" "CL05A105KA5NQNC"
 			(at 22.86 241.3 0)
 			(hide yes)
@@
 			)
 		)
-		(property "LCSC" ""
+		(property "LCSC" "C52923"
 			(at 22.86 241.3 0)
 			(hide yes)
@@
 			)
 		)
-		(property "LCSC" ""
+		(property "LCSC" "C19702"
 			(at 38.1 43.18 0)
 			(hide yes)
@@
 			)
 		)
-		(property "MPN" ""
+		(property "MPN" "CL10A106KP8NNNC"
 			(at 38.1 43.18 0)
 			(hide yes)
@@
 			)
 		)
-		(property "Characteristics" "1u 10V XR 0603"
+		(property "Characteristics" "10u 10V XR 0603"
 			(at 38.1 43.18 0)
 			(hide yes)
@@
 			)
 		)
-		(property "LCSC" ""
+		(property "LCSC" "C19702"
 			(at 38.1 73.66 0)
 			(hide yes)
@@
 			)
 		)
-		(property "MPN" ""
+		(property "MPN" "CL10A106KP8NNNC"
 			(at 38.1 73.66 0)
 			(hide yes)
@@
 			)
 		)
-		(property "Characteristics" "1u 10V XR 0603"
+		(property "Characteristics" "10u 10V XR 0603"
 			(at 38.1 73.66 0)
 			(hide yes)
@@
 			)
 		)
-		(property "MPN" "RC0805JR-100RL"
+		(property "MPN" "0805W8F0000T5E"
 			(at 304.8 55.88 0)
 			(hide yes)
@@
 			)
 		)
-		(property "LCSC" "C4143065"
+		(property "LCSC" "C17477"
 			(at 304.8 55.88 0)
 			(hide yes)
@@
 			)
 		)
-		(property "MPN" "CRG0603ZR"
+		(property "MPN" "0603WAF0000T5E"
 			(at 25.4 38.1 0)
 			(hide yes)
@@
 			)
 		)
-		(property "LCSC" "C95177"
+		(property "LCSC" "C21189"
 			(at 25.4 38.1 0)
 			(hide yes)
@@
 			)
 		)
-		(property "MPN" ""
+		(property "MPN" "CL10A106KP8NNNC"
 			(at 66.04 43.18 0)
 			(hide yes)
@@
 			)
 		)
-		(property "Characteristics" "1u 10V XR 0603"
+		(property "Characteristics" "10u 10V XR 0603"
 			(at 66.04 43.18 0)
 			(hide yes)
@@
 			)
 		)
-		(property "LCSC" ""
+		(property "LCSC" "C19702"
 			(at 66.04 43.18 0)
 			(hide yes)
@@
 			)
 		)
-		(property "MPN" "CL05A105KO5NNNC"
+		(property "MPN" "CL05A105KA5NQNC"
 			(at 33.02 241.3 0)
 			(hide yes)
@@
 			)
 		)
-		(property "LCSC" ""
+		(property "LCSC" "C52923"
 			(at 33.02 241.3 0)
 			(hide yes)
@@
 			)
 		)
-		(property "MPN" "CL05A105KO5NNNC"
+		(property "MPN" "CL05A105KA5NQNC"
 			(at 27.94 241.3 0)
 			(hide yes)
@@
 			)
 		)
-		(property "LCSC" ""
+		(property "LCSC" "C52923"
 			(at 27.94 241.3 0)
 			(hide yes)
@@
 			)
 		)
-		(property "MPN" ""
+		(property "MPN" "CL10A106KP8NNNC"
 			(at 66.04 73.66 0)
 			(hide yes)
@@
 			)
 		)
-		(property "Characteristics" "1u 10V XR 0603"
+		(property "Characteristics" "10u 10V XR 0603"
 			(at 66.04 73.66 0)
 			(hide yes)
@@
 			)
 		)
-		(property "LCSC" ""
+		(property "LCSC" "C19702"
 			(at 66.04 73.66 0)
 			(hide yes)
@@
 			)
 		)
-		(property "MPN" "CL05A105KO5NNNC"
+		(property "MPN" "CL05A105KA5NQNC"
 			(at 27.94 266.7 0)
 			(hide yes)
@@
 			)
 		)
-		(property "LCSC" ""
+		(property "LCSC" "C52923"
 			(at 27.94 266.7 0)
 			(hide yes)
@@
 			)
 		)
-		(property "MPN" "RC0805JR-100RL"
+		(property "MPN" "0805W8F0000T5E"
 			(at 307.34 81.28 0)
 			(hide yes)
@@
 			)
 		)
-		(property "LCSC" "C4143065"
+		(property "LCSC" "C17477"
 			(at 307.34 81.28 0)
 			(hide yes)
@@
 			)
 		)
-		(property "MPN" "CRG0603ZR"
+		(property "MPN" "0603WAF0000T5E"
 			(at 50.8 66.04 0)
 			(hide yes)
@@
 			)
 		)
-		(property "LCSC" "C95177"
+		(property "LCSC" "C21189"
 			(at 50.8 66.04 0)
 			(hide yes)
@@
 			)
 		)
-		(property "MPN" "CL05A105KO5NNNC"
+		(property "MPN" "CL05A105KA5NQNC"
 			(at 45.72 241.3 0)
 			(hide yes)
@@
 			)
 		)
-		(property "LCSC" ""
+		(property "LCSC" "C52923"
 			(at 45.72 241.3 0)
 			(hide yes)
@@
 			)
 		)
-		(property "MPN" "CRG0603ZR"
+		(property "MPN" "0603WAF0000T5E"
 			(at 50.8 35.56 0)
 			(hide yes)
@@
 			)
 		)
-		(property "LCSC" ""
+		(property "LCSC" "C21189"
 			(at 50.8 35.56 0)
 			(hide yes)
@@
 			)
 		)
-		(property "MPN" "CRG0603ZR"
+		(property "MPN" "0603WAF0000T5E"
 			(at 25.4 68.58 0)
 			(hide yes)
@@
 			)
 		)
-		(property "LCSC" "C95177"
+		(property "LCSC" "C21189"
 			(at 25.4 68.58 0)
 			(hide yes)
@@
 			)
 		)
-		(property "MPN" "CL05A105KO5NNNC"
+		(property "MPN" "CL05A105KA5NQNC"
 			(at 50.8 241.3 0)
 			(hide yes)
@@
 			)
 		)
-		(property "LCSC" ""
+		(property "LCSC" "C52923"
 			(at 50.8 241.3 0)
 			(hide yes)
@@
 			)
 		)
-		(property "MPN" "CL05A105KO5NNNC"
+		(property "MPN" "CL05A105KA5NQNC"
 			(at 22.86 266.7 0)
 			(hide yes)
@@
 			)
 		)
-		(property "LCSC" ""
+		(property "LCSC" "C52923"
 			(at 22.86 266.7 0)
 			(hide yes)
@@
 			)
 		)
-		(property "MPN" "RC0805JR-100RL"
+		(property "MPN" "0805W8F0000T5E"
 			(at 269.24 83.82 0)
 			(hide yes)
@@
 			)
 		)
-		(property "LCSC" "C4143065"
+		(property "LCSC" "C17477"
 			(at 269.24 83.82 0)
 			(hide yes)
